File: pcb/pcb.kicad_pcb (KiCad board)
At the start: 2 copper layers, 127.5 x 94.2 mm, 86 parts, among them J1 Conn_01x05_Male, J2 Conn_01x04_Male, SW1 SW_Push, SW10 SW_Push, SW11 SW_Push, SW12 SW_Push, SW13 SW_Push, SW14 SW_Push, SW15 SW_Push, SW16 SW_Push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

Commit message: add diodes note, bump kicad 6
Other:
- net class Default removed
